Commit message: add slam_toolbox package

File: robot_urdf/nav2/src/description/urdf_assem.urdf (robot description, URDF)
Before this commit: robot urdf_assem, 8 links, 7 joints
Links:
- removed link base_footprint
Joints:
- removed joint base_footprint_joint
- joint left_wheel_joint: origin xyz=-0.15942 0.0005 0.06705 rpy=0 1.5708 0 -> xyz=-0.15942 0.0005 0.0667 rpy=0 1.5708 0
- joint right_wheel_joint: origin xyz=0.15942 0.0005 0.06705 rpy=0 1.5708 0 -> xyz=0.15942 0.0005 0.0667 rpy=0 1.5708 0

Commit message: update slam branch

File: robot_urdf/nav2/src/description/urdf_assem.urdf (robot description, URDF)
Before this commit: robot urdf_assem, 7 links, 6 joints
Links:
- removed link lidar_link
- added link laser, mass 0.073084; collision mesh filename=package://nav2/meshes/lidar.STL; visual mesh filename=package://nav2/meshes/lidar.STL
Joints:
- removed joint lidar_joint
- added joint laser: type fixed, parent base_link, child laser, origin xyz=-0.0011383 -0.11245 0.29097 rpy=0 0 0, axis 0 0 0
