Commit message: modifying_nav2_params_add_cmd_vel

File: robot_urdf/description/lidar.xacro (robot description, xacro)
@@ -1,5 +1,5 @@
 <?xml version="1.0"?>
 <robot xmlns:xacro="http://www.ros.org/wiki/xacro" >
-    <link name="laser_frame">
+    <link name="laser">
     <inertial>
       <origin
@@ -35,5 +35,5 @@
     </collision>
   </link>
-  <joint name="laser_joint" type="fixed">
+  <joint name="laser" type="fixed">
     <origin
       xyz="-0.11245 0.0011383 0.29097"
@@ -42,12 +42,12 @@
       link="base_link" />
     <child
-      link="laser_frame" />
+      link="laser" />
     <axis
       xyz="0 0 0" />
   </joint>
-  <gazebo reference="laser_frame">
+  <gazebo reference="laser">
     <material>Gazebo/Red</material>
   </gazebo>
-  <gazebo reference="laser_frame">
+  <gazebo reference="laser">
     <sensor name="lidar" type="ray">
       <always_on>true</always_on>
@@ -79,5 +79,5 @@
         </ros>
         <output_type>sensor_msgs/LaserScan</output_type>
-        <frame_name>laser_frame</frame_name>
+        <frame_name>laser</frame_name>
       </plugin>
     </sensor>

File: robot_urdf/description/robot.urdf.xacro (robot description, xacro)
@@ -3,11 +3,11 @@
     <!-- Example link -->
     <xacro:include filename="robot_core.xacro" />
-    <xacro:arg name="use_ros2_control" default="true"/>
+    <!--  <xacro:arg name="use_ros2_control" default="true"/>
     <xacro:if value="$(arg use_ros2_control)">
     <xacro:include filename="ros2_control.xacro" />
     </xacro:if>
-    <xacro:unless value="$(arg use_ros2_control)">
+   <xacro:unless value="$(arg use_ros2_control)">
     <xacro:include filename="gazebo_control.xacro" />
-    </xacro:unless>
+    </xacro:unless> -->
     <!-- <xacro:include filename="gazebo_control.xacro" /> -->
     <xacro:include filename="lidar.xacro" />

File: robot_urdf/description/robot_core.xacro (robot description, xacro)
@@ -1,10 +1,11 @@
 <?xml version="1.0"?>
 <robot xmlns:xacro="http://www.ros.org/wiki/xacro">
+<!--<xacro:arg name="use_ros2_control" default="false"/>-->
 <!-- Base Footprint Setup -->
 <link name="base_footprint" />
 <joint name="base_footprint_joint" type="fixed">
     <origin xyz="0 0 0" rpy="0 0 0" />
-    <parent link="base_link" />
-    <child link="base_footprint" />
+    <parent link="base_footprint" />
+    <child link="base_link" />
 </joint>
 <!-- Base Link Body -->
@@ -71,5 +72,5 @@
     </collision>
 </link>
-<joint name="right_wheel_joint" type="continuous">
+<joint name="right_wheel" type="continuous">
     <origin xyz="0.0005 -0.15942 0.065" rpy="-1.5708 0 -3.1416" />
     <parent link="base_link" />
@@ -109,5 +110,5 @@
     </collision>
 </link>
-<joint name="left_wheel_joint" type="continuous">
+<joint name="left_wheel" type="continuous">
     <origin xyz="0.0005 0.15807 0.065" rpy="-1.5708 0 0" />
     <parent link="base_link" />
@@ -118,3 +119,45 @@
     <material>Gazebo/Black</material>
 </gazebo>
+<!-- <ros2_control name="HoverboardInterface" type="system">
+    <hardware>
+        <plugin>fake_components/GenericSystem</plugin>
+        <param name="state_following_command">true</param>
+    </hardware>
+    <joint name="left_wheel_joint">
+        <command_interface name="velocity">
+            <param name="min">-10</param>
+            <param name="max">10</param>
+        </command_interface>
+        <state_interface name="position" />
+        <state_interface name="velocity" />
+    </joint>
+    <joint name="right_wheel_joint">
+        <command_interface name="velocity">
+            <param name="min">-10</param>
+            <param name="max">10</param>
+        </command_interface>
+        <state_interface name="velocity" />
+        <state_interface name="position" />
+    </joint>
+</ros2_control> -->
+<transmission name="tran1">
+    <type>transmission_interface/SimpleTransmission</type>
+    <joint name="right_wheel_joint">
+      <hardwareInterface>hardware_interface/VelocityJointInterface</hardwareInterface>
+    </joint>
+    <actuator name="motor1">
+       <hardwareInterface>hardware_interface/VelocityJointInterface</hardwareInterface>
+     <mechanicalReduction>1</mechanicalReduction>
+    </actuator>
+  </transmission>
+  <transmission name="tran2">
+    <type>transmission_interface/SimpleTransmission</type>
+    <joint name="left_wheel_joint">
+      <hardwareInterface>hardware_interface/VelocityJointInterface</hardwareInterface>
+    </joint>
+    <actuator name="motor2">
+      <hardwareInterface>hardware_interface/VelocityJointInterface</hardwareInterface>
+      <mechanicalReduction>1</mechanicalReduction>
+    </actuator>
+  </transmission>
 </robot>

File: robot_urdf/description/ros2_control.xacro (robot description, xacro)
@@ -1,4 +1,37 @@
 <?xml version="1.0"?>
 <robot xmlns:xacro="http://www.ros.org/wiki/xacro">
+    <!-- <ros2_control name="GazeboSystem" type="system">
+        <hardware>
+            <plugin>gazebo_ros2_control/GazeboSystem</plugin>
+        </hardware>
+        <joint name="left_wheel_joint">
+            <command_interface name="velocity">
+                <param name="min">-10</param>
+                <param name="max">10</param>
+            </command_interface>
+            <state_interface name="position" />
+                <param name="max">10</param>
+            </command_interface>
+            <state_interface name="velocity" />
+            <state_interface name="position" />
+        </joint>
+    </ros2_control>
+    <gazebo>
+        <plugin filename="libgazebo_ros2_control.so" name="gazebo_ros2_control">
+            <parameters>$(find navigation_control)/config/my_controllers.yaml</parameters>
+        </plugin>
+    </gazebo>          <command_interface name="velocity">
+                <param name="min">-10</param>
+                <param name="max">10</param>
+            </command_interface>
+            <state_interface name="velocity" />
+            <state_interface name="position" />
+        </joint>
+    </ros2_control>
+    <gazebo>
+        <plugin filename="libgazebo_ros2_control.so" name="gazebo_ros2_control">
+            <parameters>$(find navigation_control)/config/my_controllers.yaml</parameters>
+        </plugin>
+    </gazebo> -->
     <ros2_control name="GazeboSystem" type="system">
         <hardware>
